Commit message: added camera

File: src/robot_bringup/urdf/rc_car.urdf.xacro (robot description, xacro)
@@ -193,4 +193,28 @@
   </joint>
   <!-- ================================================================== -->
+  <!-- RGB camera sensor                                                   -->
+  <!-- ================================================================== -->
+  <link name="camera_link">
+    <visual>
+      <geometry>
+        <box size="0.06 0.04 0.04"/>
+      </geometry>
+      <material name="blue">
+        <color rgba="0.1 0.1 0.9 1.0"/>
+      </material>
+    </visual>
+    <collision>
+      <geometry>
+        <box size="0.06 0.04 0.04"/>
+      </geometry>
+    </collision>
+    <xacro:box_inertia m="0.03" x="0.06" y="0.04" z="0.04"/>
+  </link>
+  <joint name="camera_joint" type="fixed">
+    <parent link="chassis"/>
+    <child  link="camera_link"/>
+    <origin xyz="${wheelbase + 0.03} 0 ${body_height + 0.02}" rpy="0 0 0"/>
+  </joint>
+  <!-- ================================================================== -->
   <!-- Gazebo plugins                                                      -->
   <!-- ================================================================== -->
@@ -265,3 +289,24 @@
     </sensor>
   </gazebo>
+  <!-- RGB camera sensor (bridged with ros_gz_bridge) -->
+  <gazebo reference="camera_link">
+    <sensor name="rgb_camera" type="camera">
+      <always_on>true</always_on>
+      <visualize>true</visualize>
+      <update_rate>30</update_rate>
+      <topic>/camera/image_raw</topic>
+      <camera>
+        <horizontal_fov>1.3962634</horizontal_fov>
+        <image>
+          <width>640</width>
+          <height>480</height>
+          <format>R8G8B8</format>
+        </image>
+        <clip>
+          <near>0.1</near>
+          <far>50.0</far>
+        </clip>
+      </camera>
+    </sensor>
+  </gazebo>
 </robot>

Commit message: fixed wheel inversion

File: src/robot_bringup/urdf/rc_car.urdf.xacro (robot description, xacro)
@@ -67,5 +67,5 @@
            axis aligns with the vehicle lateral axis. -->
       <origin xyz="${x} ${y} 0" rpy="${pi/2} 0 0"/>
-      <axis xyz="0 0 1"/>
+      <axis xyz="0 0 -1"/>
     </joint>
   </xacro:macro>
@@ -109,5 +109,5 @@
       <child  link="${name}"/>
       <origin xyz="0 0 0" rpy="${pi/2} 0 0"/>
-      <axis xyz="0 0 1"/>
+      <axis xyz="0 0 -1"/>
     </joint>
   </xacro:macro>

Commit message: mounted lidar higher

File: src/robot_bringup/urdf/rc_car.urdf.xacro (robot description, xacro)
@@ -179,5 +179,5 @@
     <child  link="lidar_link"/>
     <!-- Mount the LiDAR on top of the chassis, towards the front. -->
-    <origin xyz="${wheelbase*0.6} 0 ${body_height + 0.03}" rpy="0 0 0"/>
+    <origin xyz="${wheelbase*0.6} 0 ${body_height + 0.06}" rpy="0 0 0"/>
   </joint>
   <!-- ================================================================== -->
